Commit message: modified the urdf model of the robot, created wheel links and joints

File: urdf/my_robot.xacro (robot description, xacro)
@@ -1,2 +1,3 @@
+<?xml version='1.0'?>
 <robot name="my_robot" xmlns:xacro="http://www.ros.org/wiki/xacro">
   <link name="robot_footprint"></link>
@@ -54,3 +55,65 @@
     </visual>
   </link>
+  <link name="left_wheel">
+    <collision name="left_wheel_collision">
+      <origin xyz="0 0 0" rpy=" 0 1.5707 1.5707"/>
+      <geometry>
+        <cylinder radius="0.1" length="0.05"/>
+      </geometry>
+    </collision>
+    <inertial>
+      <mass value="5.0"/>
+      <origin xyz="0 0 0" rpy=" 0 1.5707 1.5707"/>
+      <inertia
+          ixx="0.1" ixy="0" ixz="0"
+          iyy="0.1" iyz="0"
+          izz="0.1"
+      />
+    </inertial>
+    <visual name='left_wheel_visual'>
+      <origin xyz="0 0 0" rpy=" 0 1.5707 1.5707"/>
+      <geometry>
+        <cylinder radius="0.1" length="0.05"/>
+      </geometry>
+    </visual>
+  </link>
+  <link name="right_wheel">
+    <collision name="left_wheel_collision">
+      <origin xyz="0 0 0" rpy=" 0 1.5707 1.5707"/>
+      <geometry>
+        <cylinder radius="0.1" length="0.05"/>
+      </geometry>
+    </collision>
+    <inertial>
+      <mass value="5.0"/>
+      <origin xyz="0 0 0" rpy=" 0 1.5707 1.5707"/>
+      <inertia
+          ixx="0.1" ixy="0" ixz="0"
+          iyy="0.1" iyz="0"
+          izz="0.1"
+      />
+    </inertial>
+    <visual name='right_wheel_visual'>
+      <origin xyz="0 0 0" rpy=" 0 1.5707 1.5707"/>
+      <geometry>
+        <cylinder radius="0.1" length="0.05"/>
+      </geometry>
+    </visual>
+  </link>
+  <joint type="continuous" name="left_wheel_hinge">
+    <origin xyz="0 0.15 0" rpy="0 0 0"/>
+    <child link="left_wheel"/>
+    <parent link="chassis"/>
+    <axis xyz="0 1 0" rpy="0 0 0"/>
+    <limit effort="10000" velocity="1000"/>
+    <dynamics damping="1.0" friction="1.0"/>
+  </joint>
+  <joint type="continuous" name="right_wheel_hinge">
+    <origin xyz="0 -0.15 0" rpy="0 0 0"/>
+    <child link="right_wheel"/>
+    <parent link="chassis"/>
+    <axis xyz="0 1 0" rpy="0 0 0"/>
+    <limit effort="10000" velocity="1000"/>
+    <dynamics damping="1.0" friction="1.0"/>
+  </joint>
 </robot>

Commit message: added urdf camera link and joint to the robot

File: urdf/my_robot.xacro (robot description, xacro)
@@ -117,3 +117,32 @@
     <dynamics damping="1.0" friction="1.0"/>
   </joint>
+  <link name="camera">
+    <visual>
+      <origin xyz="0 0 0" rpy="0 0 0"/>
+      <geometry>
+        <box size="0.05 0.05 0.05"/>
+      </geometry>
+    </visual>
+    <collision name="camera_collision">
+      <origin xyz="0 0 0" rpy=" 0 0 0"/>
+      <geometry>
+        <box size="0.05 0.05 0.05"/>
+      </geometry>
+    </collision>
+    <inertial>
+      <mass value="0.1"/>
+      <origin xyz="0 0 0" rpy=" 0 0 0"/>
+      <inertia
+          ixx="1e-6" ixy="0" ixz="0"
+          iyy="1e-6" iyz="0"
+          izz="1e-6"
+      />
+    </inertial>
+  </link>
+  <joint type="fixed" name="camera_joint">
+    <origin xyz="0.2 0 0" rpy="0 0 0"/>
+    <child link="camera"/>
+    <parent link="chassis"/>
+    <axis xyz="0 1 0"/>
+  </joint>
 </robot>

Commit message: added camera and lidar to urdf model

File: urdf/my_robot.xacro (robot description, xacro)
@@ -118,10 +118,4 @@
   </joint>
   <link name="camera">
-    <visual>
-      <origin xyz="0 0 0" rpy="0 0 0"/>
-      <geometry>
-        <box size="0.05 0.05 0.05"/>
-      </geometry>
-    </visual>
     <collision name="camera_collision">
       <origin xyz="0 0 0" rpy=" 0 0 0"/>
@@ -139,4 +133,10 @@
       />
     </inertial>
+    <visual>
+      <origin xyz="0 0 0" rpy="0 0 0"/>
+      <geometry>
+        <box size="0.05 0.05 0.05"/>
+      </geometry>
+    </visual>
   </link>
   <joint type="fixed" name="camera_joint">
@@ -146,3 +146,32 @@
     <axis xyz="0 1 0"/>
   </joint>
+  <link name="hokuyo">
+    <collision name="hokuyo_collision">
+      <origin xyz="0 0 0" rpy=" 0 0 0"/>
+      <geometry>
+        <box size="0.1 0.1 0.1"/>
+      </geometry>
+    </collision>
+    <inertial>
+      <mass value="1e-5"/>
+      <origin xyz="0 0 0" rpy=" 0 0 0"/>
+      <inertia
+          ixx="1e-6" ixy="0" ixz="0"
+          iyy="1e-6" iyz="0"
+          izz="1e-6"
+      />
+    </inertial>
+    <visual>
+      <origin xyz="0 0 0" rpy="0 0 0"/>
+      <geometry>
+        <mesh filename="package://my_robot/meshes/hokuyo.dae"/>
+      </geometry>
+    </visual>
+  </link>
+  <joint name="hokuyo_joint" type="fixed">
+    <axis xyz="0 1 0"/>
+    <origin xyz="0.15 0 0.1" rpy=" 0 0 0"/>
+    <parent link="chassis"/>
+    <child link="hokuyo"/>
+  </joint>
 </robot>

Commit message: added colout and fixed adjusted the hokoyu joint origin to better fit to the base

File: urdf/my_robot.xacro (robot description, xacro)
@@ -148,5 +148,4 @@
   <link name="hokuyo">
     <collision name="hokuyo_collision">
-      <origin xyz="0 0 0" rpy=" 0 0 0"/>
       <geometry>
         <box size="0.1 0.1 0.1"/>
@@ -162,6 +161,5 @@
       />
     </inertial>
-    <visual>
-      <origin xyz="0 0 0" rpy="0 0 0"/>
+    <visual name="hokuyo_mesh_visual">
       <geometry>
         <mesh filename="package://my_robot/meshes/hokuyo.dae"/>
@@ -170,8 +168,20 @@
   </link>
   <joint name="hokuyo_joint" type="fixed">
+    <origin xyz="0.15 0 0.085" rpy=" 0 0 0"/>
     <axis xyz="0 1 0"/>
-    <origin xyz="0.15 0 0.1" rpy=" 0 0 0"/>
     <parent link="chassis"/>
     <child link="hokuyo"/>
   </joint>
+  <gazebo reference="left_wheel">
+    <material>Gazebo/Red</material>
+  </gazebo>
+  <gazebo reference="right_wheel">
+    <material>Gazebo/Red</material>
+  </gazebo>
+  <gazebo reference="chassis">
+    <material>Gazebo/Green</material>
+  </gazebo>
+  <gazebo reference="camera">
+    <material>Gazebo/Blue</material>
+  </gazebo>
 </robot>
